Commit message: Current Update
Updated the current version

File: kit1_spider.urdf (robot description, URDF)
Before this commit: robot spider_bot, 25 links, 24 joints
Joints:
- joint leg0_joint0: axis 0 0 1 -> 0 0 -1
- joint leg1_joint0: axis 0 0 1 -> 0 0 -1
- joint leg2_joint0: axis 0 0 1 -> 0 0 -1
- joint leg3_joint0: axis 0 0 1 -> 0 0 -1
